File: Skripsie/Skripsie.sch (KiCad schematic (older format))
At the start: 262 parts, among them J1 STM32F4_Discovery, U1 SN74HC595, U2 SN74HC595, U3 TPIC6C596, U4 SN74HC595, U5 SN74HC595

Commit message: Updated Schematic
Parts:
- added C1, C2: 47pF, Capacitor_SMD:C_0805_2012Metric_Pad1.15x1.40mm_HandSolder, symbol Device:C
- added C3: 10nF, Capacitor_SMD:C_0805_2012Metric_Pad1.15x1.40mm_HandSolder, symbol Device:C
- added C4: 1nF, Capacitor_SMD:C_0805_2012Metric_Pad1.15x1.40mm_HandSolder, symbol Device:C
- added C5: 100nF, Capacitor_SMD:C_0805_2012Metric_Pad1.15x1.40mm_HandSolder, symbol Device:C
- added J2: USB_B, Connector_USB:USB_B_OST_USB-B1HSxx_Horizontal, symbol Connector:USB_B
- added LCD1: PC1601A, Connector_PinHeader_2.54mm:PinHeader_1x16_P2.54mm_Vertical, symbol Pieter:PC1601A
- added POT1, POT2: 10kE, digikey-footprints:Trimpot_3.8mmx3.6mm_TC33X-2-103E, symbol dk_Trimmer-Potentiometers:TC33X-2-103E
- added R17, R18: R, Resistor_SMD:R_0805_2012Metric_Pad1.15x1.40mm_HandSolder, symbol Device:R
- added R19, R20: 27E, Resistor_SMD:R_0805_2012Metric_Pad1.15x1.40mm_HandSolder, symbol Device:R
- added R21, R22: 1K, Resistor_SMD:R_0805_2012Metric_Pad1.15x1.40mm_HandSolder, symbol Device:R
- added R23: 1M, Resistor_SMD:R_0805_2012Metric_Pad1.15x1.40mm_HandSolder, symbol Device:R
- added U6: FT230XS-U, digikey-footprints:SSOP-16_W3.90mm, symbol dk_Interface-Controllers:FT230XS-U
- renumbered R13 to R10, R6 to R11, R14 to R12, R7 to R13, R15 to R14, R8 to R15, R9 to R2, R2 to R3, R10 to R4, R3 to R5, R11 to R6, R4 to R7, R12 to R8, R5 to R9, U4 to U2, U2 to U3, U5 to U4, U3 to U5
Connections:
- net labels added: +3V3, ADC_TEMPO, ADC_VOLUME, BTN_R0, BTN_R1, BTN_R2, BTN_R3, BTN_R4, BTN_RCLK, BTN_SRCLK, LCD_DB4, LCD_DB5, LCD_DB6, LCD_DB7, LCD_E, LCD_RNW, LCD_RS, LED_RCLK, LED_SRCLK, USART1_RX, USART1_TX
- net labels removed: BTN_REG_CLK, BTN_SHFT_REG_CLK, LED_REGCLK, LED_SHIFT_REG_CLK, br0, br1, br2, br3, br4
- wire segments 583 -> 640
- no-connect marks 0 -> 71
Other:
- note added: "16x5 BUTTON MATRIX"
- note added: "16x5 LED MATRIX"
- note added: "BUTTON DRIVER"
- note added: "LCD"
- note added: "LED DRIVER"
- note added: "POTS"
- note added: "SERIAL TO USB\n(OPTIONAL)"
- note added: "STM32F4-DISCOVERY"

Commit message: Corrected LED Driver circuit for REV A
Parts:
- removed U3: SN74HC595, Package_SO:SOIC-16_3.9x9.9mm_P1.27mm, symbol Pieter:SN74HC595
- added U?: TPIC6C596, Package_SO:SOIC-16_3.9x9.9mm_P1.27mm, symbol Pieter:TPIC6C596
Connections:
- no-connect marks 71 -> 70

Commit message: Altered LED Driver and Button driver circuits - Rev B
Parts:
- removed R10, R11, R12, R13, R14, R15, R16, R6, R7, R8, R9: R, Resistor_SMD:R_0805_2012Metric_Pad1.15x1.40mm_HandSolder, symbol Device:R
- removed U2: SN74HC595, Package_SO:SOIC-16_3.9x9.9mm_P1.27mm, symbol Pieter:SN74HC595
- removed U5, U?: TPIC6C596, Package_SO:SOIC-16_3.9x9.9mm_P1.27mm, symbol Pieter:TPIC6C596
- added Q1, Q2: ULN2803ADWR, digikey-footprints:SOIC-18_W7.5mm, symbol dk_Transistors-Bipolar-BJT-Arrays:ULN2803ADWR
- added U2, U5: 4017, symbol 4xxx:4017
- added U3: SN74HC08N, digikey-footprints:DIP-14_W3mm, symbol dk_Logic-Gates-and-Inverters:SN74HC08N
- added U6: SN74HC595, Package_SO:SOIC-16_3.9x9.9mm_P1.27mm, symbol Pieter:SN74HC595
- renumbered R21 to R10, R22 to R11, R23 to R12, R17 to R6, R18 to R7, R19 to R8, R20 to R9, U6 to U7
Connections:
- wire segments 640 -> 629
- no-connect marks 70 -> 85

Commit message: Added new pinout file & reset mechanism for Button driver
Parts:
- added D?: DIODE, Diode_SMD:D_0805_2012Metric_Pad1.15x1.40mm_HandSolder, symbol pspice:DIODE
Connections:
- net labels added: BTN_RESET
- net labels removed: BTN_RCLK
- wire segments 629 -> 633
Changed lines of the file:
@@
 F 3 "" H 7900 1650 50  0001 C CNN
 	1    7900 1650
-	0    -1   -1   0
+	1    0    0    -1
 $EndComp
 $Comp
@@
 BTN_R3
 Text GLabel 4050 9600 0    50   Input ~ 0
-BTN_RCLK
+BTN_RESET
 Text GLabel 4800 9600 2    50   Input ~ 0
 BTN_SRCLK
@@
 U 1 1 5F25C8C3
 P 7900 2450
-F 0 "U2" H 7900 3428 50  0000 C CNN
-F 1 "4017" H 7900 3337 50  0000 C CNN
+F 0 "U2" H 7650 3100 50  0000 C CNN
+F 1 "4017" H 8100 3100 50  0000 C CNN
 F 2 "" H 7900 2450 50  0001 C CNN
 F 3 "http://www.intersil.com/content/dam/Intersil/documents/cd40/cd4017bms-22bms.pdf" H 7900 2450 50  0001 C CNN
@@
 U 1 1 5F25D6DC
 P 7950 4500
-F 0 "U5" H 7950 5478 50  0000 C CNN
-F 1 "4017" H 7950 5387 50  0000 C CNN
+F 0 "U5" H 7700 5150 50  0000 C CNN
+F 1 "4017" H 8150 5150 50  0000 C CNN
 F 2 "" H 7950 4500 50  0001 C CNN
 F 3 "http://www.intersil.com/content/dam/Intersil/documents/cd40/cd4017bms-22bms.pdf" H 7950 4500 50  0001 C CNN
@@
 F 3 "" H 7950 3700 50  0001 C CNN
 	1    7950 3700
-	0    -1   -1   0
+	0    1    1    0
 $EndComp
 $Comp
@@
 	7450 4100 7300 4100
 Wire Wire Line
-	7150 4100 7150 2250
-Wire Wire Line
 	7150 2250 7400 2250
 Wire Wire Line
@@
 	1    0    0    -1
 $EndComp
+$Comp
+L pspice:DIODE D?
+U 1 1 5C85A292
+P 7150 3700
+F 0 "D?" V 7196 3572 50  0000 R CNN
+F 1 "DIODE" V 7105 3572 50  0000 R CNN
+F 2 "Diode_SMD:D_0805_2012Metric_Pad1.15x1.40mm_HandSolder" H 7150 3700 50  0001 C CNN
+F 3 "" H 7150 3700 50  0001 C CNN
+	1    7150 3700
+	0    -1   -1   0
+$EndComp
+Wire Wire Line
+	7150 4100 7150 3900
+Wire Wire Line
+	7150 3500 7150 2250
+Wire Wire Line
+	7150 2250 6200 2250
+Wire Wire Line
+	6200 2250 6200 1850
+Wire Wire Line
+	6200 1850 5950 1850
+Connection ~ 7150 2250
+Text GLabel 5950 1850 0    50   Input ~ 0
+BTN_RESET
 $EndSCHEMATC

Commit message: Corrected Diode orientation
Parts:
- removed U3: SN74HC08N, digikey-footprints:DIP-14_W3mm, symbol dk_Logic-Gates-and-Inverters:SN74HC08N
- added R? (x5): R, Resistor_SMD:R_0805_2012Metric_Pad1.15x1.40mm_HandSolder, symbol Device:R
- added U?: SN74LVC1G08, symbol Pieter:SN74LVC1G08
Connections:
- wire segments 633 -> 638
- no-connect marks 85 -> 76

Commit message: Updated the schematic and ordered parts
Parts:
- removed C5: 100nF, Capacitor_SMD:C_0805_2012Metric_Pad1.15x1.40mm_HandSolder, symbol Device:C
- removed R7: R, Resistor_SMD:R_0805_2012Metric_Pad1.15x1.40mm_HandSolder, symbol Device:R
- removed U?: SN74LVC1G08, symbol Pieter:SN74LVC1G08
- added C1, C2, C3: 10nF, Capacitor_SMD:C_1206_3216Metric_Pad1.42x1.75mm_HandSolder, symbol Device:C
- added J10: LED_R_TEST, Connector_PinHeader_2.54mm:PinHeader_1x05_P2.54mm_Vertical, symbol Connector_Generic:Conn_01x05
- added J11: 3V3, Connector_PinHeader_2.54mm:PinHeader_1x01_P2.54mm_Vertical, symbol Connector_Generic:Conn_01x01
- added J12: UART_TEST, Connector_PinHeader_2.54mm:PinHeader_1x02_P2.54mm_Vertical, symbol Connector_Generic:Conn_01x02
- added J2: LCD_TEST, Connector_PinHeader_2.54mm:PinHeader_1x07_P2.54mm_Vertical, symbol Connector_Generic:Conn_01x07
- added J3: BTN_C_TEST, Connector_PinHeader_2.54mm:PinHeader_1x16_P2.54mm_Vertical, symbol Connector_Generic:Conn_01x16
- added J4: LED_C_TEST, Connector_PinHeader_2.54mm:PinHeader_1x16_P2.54mm_Vertical, symbol Connector_Generic:Conn_01x16
- added J5: LED_SER_TEST, Connector_PinHeader_2.54mm:PinHeader_1x03_P2.54mm_Vertical, symbol Connector_Generic:Conn_01x03
- added J6: BTN_SER_TEST, Connector_PinHeader_2.54mm:PinHeader_1x02_P2.54mm_Vertical, symbol Connector_Generic:Conn_01x02
- added J7: GND, Connector_PinHeader_2.54mm:PinHeader_1x01_P2.54mm_Vertical, symbol Connector_Generic:Conn_01x01
- added J8: 5V, Connector_PinHeader_2.54mm:PinHeader_1x01_P2.54mm_Vertical, symbol Connector_Generic:Conn_01x01
- added J9: BTN_R_TEST, Connector_PinHeader_2.54mm:PinHeader_1x05_P2.54mm_Vertical, symbol Connector_Generic:Conn_01x05
- added POT3: 20KE, Potentiometer_SMD:Potentiometer_Bourns_3314G_Vertical, symbol dk_Trimmer-Potentiometers:TC33X-2-103E
- added U4: SN74HC08N, Package_SO:SOIC-14_3.9x8.7mm_P1.27mm, symbol dk_Logic-Gates-and-Inverters:SN74HC08N
- C4: renamed from C2; footprint Capacitor_SMD:C_0805_2012Metric_Pad1.15x1.40mm_HandSolder -> Capacitor_SMD:C_1206_3216Metric_Pad1.42x1.75mm_HandSolder
- C5: renamed from C1; footprint Capacitor_SMD:C_0805_2012Metric_Pad1.15x1.40mm_HandSolder -> Capacitor_SMD:C_1206_3216Metric_Pad1.42x1.75mm_HandSolder
- C6: renamed from C3; footprint Capacitor_SMD:C_0805_2012Metric_Pad1.15x1.40mm_HandSolder -> Capacitor_SMD:C_1206_3216Metric_Pad1.42x1.75mm_HandSolder
- C7: renamed from C4; footprint Capacitor_SMD:C_0805_2012Metric_Pad1.15x1.40mm_HandSolder -> Capacitor_SMD:C_1206_3216Metric_Pad1.42x1.75mm_HandSolder
- D1, D10, D11, D12, D13, D14, D15, D16, D17, D18, D19, D2, D20, D21, D22, D23, D24, D25, D26, D27, D28, D29, D3, D30, D31, D32, D4, D5, D6, D7, D8, D9: value LED -> LTST-C150KFKT; footprint LED_SMD:LED_Cree-PLCC4_3.2x2.8mm_CCW -> LED_SMD:LED_1206_3216Metric_Pad1.42x1.75mm_HandSolder
- D100: renamed from D99; value DIODE -> FDLL4148; footprint Diode_SMD:D_0805_2012Metric_Pad1.15x1.40mm_HandSolder -> Diode_SMD:D_MiniMELF_Handsoldering
- D101: renamed from D100; value DIODE -> FDLL4148; footprint Diode_SMD:D_0805_2012Metric_Pad1.15x1.40mm_HandSolder -> Diode_SMD:D_MiniMELF_Handsoldering
- D102: renamed from D101; value DIODE -> FDLL4148; footprint Diode_SMD:D_0805_2012Metric_Pad1.15x1.40mm_HandSolder -> Diode_SMD:D_MiniMELF_Handsoldering
- D103: renamed from D102; value DIODE -> FDLL4148; footprint Diode_SMD:D_0805_2012Metric_Pad1.15x1.40mm_HandSolder -> Diode_SMD:D_MiniMELF_Handsoldering
- D104: renamed from D103; value DIODE -> FDLL4148; footprint Diode_SMD:D_0805_2012Metric_Pad1.15x1.40mm_HandSolder -> Diode_SMD:D_MiniMELF_Handsoldering
- D105: renamed from D104; value DIODE -> FDLL4148; footprint Diode_SMD:D_0805_2012Metric_Pad1.15x1.40mm_HandSolder -> Diode_SMD:D_MiniMELF_Handsoldering
- D106: renamed from D105; value DIODE -> FDLL4148; footprint Diode_SMD:D_0805_2012Metric_Pad1.15x1.40mm_HandSolder -> Diode_SMD:D_MiniMELF_Handsoldering
- D107: renamed from D106; value DIODE -> FDLL4148; footprint Diode_SMD:D_0805_2012Metric_Pad1.15x1.40mm_HandSolder -> Diode_SMD:D_MiniMELF_Handsoldering
- D108: renamed from D107; value DIODE -> FDLL4148; footprint Diode_SMD:D_0805_2012Metric_Pad1.15x1.40mm_HandSolder -> Diode_SMD:D_MiniMELF_Handsoldering
- D109: renamed from D108; value DIODE -> FDLL4148; footprint Diode_SMD:D_0805_2012Metric_Pad1.15x1.40mm_HandSolder -> Diode_SMD:D_MiniMELF_Handsoldering
- D110: renamed from D109; value DIODE -> FDLL4148; footprint Diode_SMD:D_0805_2012Metric_Pad1.15x1.40mm_HandSolder -> Diode_SMD:D_MiniMELF_Handsoldering
- D111: renamed from D110; value DIODE -> FDLL4148; footprint Diode_SMD:D_0805_2012Metric_Pad1.15x1.40mm_HandSolder -> Diode_SMD:D_MiniMELF_Handsoldering
- D112: renamed from D111; value DIODE -> FDLL4148; footprint Diode_SMD:D_0805_2012Metric_Pad1.15x1.40mm_HandSolder -> Diode_SMD:D_MiniMELF_Handsoldering
- D113: renamed from D112; value DIODE -> FDLL4148; footprint Diode_SMD:D_0805_2012Metric_Pad1.15x1.40mm_HandSolder -> Diode_SMD:D_MiniMELF_Handsoldering
- D114: renamed from D113; value DIODE -> FDLL4148; footprint Diode_SMD:D_0805_2012Metric_Pad1.15x1.40mm_HandSolder -> Diode_SMD:D_MiniMELF_Handsoldering
- D115: renamed from D114; value DIODE -> FDLL4148; footprint Diode_SMD:D_0805_2012Metric_Pad1.15x1.40mm_HandSolder -> Diode_SMD:D_MiniMELF_Handsoldering
- D116: renamed from D115; value DIODE -> FDLL4148; footprint Diode_SMD:D_0805_2012Metric_Pad1.15x1.40mm_HandSolder -> Diode_SMD:D_MiniMELF_Handsoldering
- D117: renamed from D116; value DIODE -> FDLL4148; footprint Diode_SMD:D_0805_2012Metric_Pad1.15x1.40mm_HandSolder -> Diode_SMD:D_MiniMELF_Handsoldering
- D118: renamed from D117; value DIODE -> FDLL4148; footprint Diode_SMD:D_0805_2012Metric_Pad1.15x1.40mm_HandSolder -> Diode_SMD:D_MiniMELF_Handsoldering
- D119: renamed from D118; value DIODE -> FDLL4148; footprint Diode_SMD:D_0805_2012Metric_Pad1.15x1.40mm_HandSolder -> Diode_SMD:D_MiniMELF_Handsoldering
- D120: renamed from D119; value DIODE -> FDLL4148; footprint Diode_SMD:D_0805_2012Metric_Pad1.15x1.40mm_HandSolder -> Diode_SMD:D_MiniMELF_Handsoldering
- D121: renamed from D120; value DIODE -> FDLL4148; footprint Diode_SMD:D_0805_2012Metric_Pad1.15x1.40mm_HandSolder -> Diode_SMD:D_MiniMELF_Handsoldering
- D122: renamed from D121; value DIODE -> FDLL4148; footprint Diode_SMD:D_0805_2012Metric_Pad1.15x1.40mm_HandSolder -> Diode_SMD:D_MiniMELF_Handsoldering
- D123: renamed from D122; value DIODE -> FDLL4148; footprint Diode_SMD:D_0805_2012Metric_Pad1.15x1.40mm_HandSolder -> Diode_SMD:D_MiniMELF_Handsoldering
- D124: renamed from D123; value DIODE -> FDLL4148; footprint Diode_SMD:D_0805_2012Metric_Pad1.15x1.40mm_HandSolder -> Diode_SMD:D_MiniMELF_Handsoldering
- D125: renamed from D124; value DIODE -> FDLL4148; footprint Diode_SMD:D_0805_2012Metric_Pad1.15x1.40mm_HandSolder -> Diode_SMD:D_MiniMELF_Handsoldering
- D126: renamed from D125; value DIODE -> FDLL4148; footprint Diode_SMD:D_0805_2012Metric_Pad1.15x1.40mm_HandSolder -> Diode_SMD:D_MiniMELF_Handsoldering
- D127: renamed from D126; value DIODE -> FDLL4148; footprint Diode_SMD:D_0805_2012Metric_Pad1.15x1.40mm_HandSolder -> Diode_SMD:D_MiniMELF_Handsoldering
- D128: renamed from D127; value DIODE -> FDLL4148; footprint Diode_SMD:D_0805_2012Metric_Pad1.15x1.40mm_HandSolder -> Diode_SMD:D_MiniMELF_Handsoldering
- D129: renamed from D128; value DIODE -> FDLL4148; footprint Diode_SMD:D_0805_2012Metric_Pad1.15x1.40mm_HandSolder -> Diode_SMD:D_MiniMELF_Handsoldering
- D130: renamed from D129; value DIODE -> FDLL4148; footprint Diode_SMD:D_0805_2012Metric_Pad1.15x1.40mm_HandSolder -> Diode_SMD:D_MiniMELF_Handsoldering
- D131: renamed from D130; value DIODE -> FDLL4148; footprint Diode_SMD:D_0805_2012Metric_Pad1.15x1.40mm_HandSolder -> Diode_SMD:D_MiniMELF_Handsoldering
- D132: renamed from D131; value DIODE -> FDLL4148; footprint Diode_SMD:D_0805_2012Metric_Pad1.15x1.40mm_HandSolder -> Diode_SMD:D_MiniMELF_Handsoldering
- D133: renamed from D132; value DIODE -> FDLL4148; footprint Diode_SMD:D_0805_2012Metric_Pad1.15x1.40mm_HandSolder -> Diode_SMD:D_MiniMELF_Handsoldering
- D134: renamed from D133; value DIODE -> FDLL4148; footprint Diode_SMD:D_0805_2012Metric_Pad1.15x1.40mm_HandSolder -> Diode_SMD:D_MiniMELF_Handsoldering
- D135: renamed from D134; value DIODE -> FDLL4148; footprint Diode_SMD:D_0805_2012Metric_Pad1.15x1.40mm_HandSolder -> Diode_SMD:D_MiniMELF_Handsoldering
- D136: renamed from D135; value DIODE -> FDLL4148; footprint Diode_SMD:D_0805_2012Metric_Pad1.15x1.40mm_HandSolder -> Diode_SMD:D_MiniMELF_Handsoldering
- D137: renamed from D136; value DIODE -> FDLL4148; footprint Diode_SMD:D_0805_2012Metric_Pad1.15x1.40mm_HandSolder -> Diode_SMD:D_MiniMELF_Handsoldering
- D138: renamed from D137; value DIODE -> FDLL4148; footprint Diode_SMD:D_0805_2012Metric_Pad1.15x1.40mm_HandSolder -> Diode_SMD:D_MiniMELF_Handsoldering
- D139: renamed from D138; value DIODE -> FDLL4148; footprint Diode_SMD:D_0805_2012Metric_Pad1.15x1.40mm_HandSolder -> Diode_SMD:D_MiniMELF_Handsoldering
- D140: renamed from D139; value DIODE -> FDLL4148; footprint Diode_SMD:D_0805_2012Metric_Pad1.15x1.40mm_HandSolder -> Diode_SMD:D_MiniMELF_Handsoldering
- D141: renamed from D140; value DIODE -> FDLL4148; footprint Diode_SMD:D_0805_2012Metric_Pad1.15x1.40mm_HandSolder -> Diode_SMD:D_MiniMELF_Handsoldering
- D142: renamed from D141; value DIODE -> FDLL4148; footprint Diode_SMD:D_0805_2012Metric_Pad1.15x1.40mm_HandSolder -> Diode_SMD:D_MiniMELF_Handsoldering
- D143: renamed from D142; value DIODE -> FDLL4148; footprint Diode_SMD:D_0805_2012Metric_Pad1.15x1.40mm_HandSolder -> Diode_SMD:D_MiniMELF_Handsoldering
- D144: renamed from D143; value DIODE -> FDLL4148; footprint Diode_SMD:D_0805_2012Metric_Pad1.15x1.40mm_HandSolder -> Diode_SMD:D_MiniMELF_Handsoldering
- D145: renamed from D144; value DIODE -> FDLL4148; footprint Diode_SMD:D_0805_2012Metric_Pad1.15x1.40mm_HandSolder -> Diode_SMD:D_MiniMELF_Handsoldering
- D146: renamed from D145; value DIODE -> FDLL4148; footprint Diode_SMD:D_0805_2012Metric_Pad1.15x1.40mm_HandSolder -> Diode_SMD:D_MiniMELF_Handsoldering
- D147: renamed from D146; value DIODE -> FDLL4148; footprint Diode_SMD:D_0805_2012Metric_Pad1.15x1.40mm_HandSolder -> Diode_SMD:D_MiniMELF_Handsoldering
- D148: renamed from D147; value DIODE -> FDLL4148; footprint Diode_SMD:D_0805_2012Metric_Pad1.15x1.40mm_HandSolder -> Diode_SMD:D_MiniMELF_Handsoldering
- D149: renamed from D148; value DIODE -> FDLL4148; footprint Diode_SMD:D_0805_2012Metric_Pad1.15x1.40mm_HandSolder -> Diode_SMD:D_MiniMELF_Handsoldering
- D150: renamed from D149; value DIODE -> FDLL4148; footprint Diode_SMD:D_0805_2012Metric_Pad1.15x1.40mm_HandSolder -> Diode_SMD:D_MiniMELF_Handsoldering
- D151: renamed from D150; value DIODE -> FDLL4148; footprint Diode_SMD:D_0805_2012Metric_Pad1.15x1.40mm_HandSolder -> Diode_SMD:D_MiniMELF_Handsoldering
- D152: renamed from D151; value DIODE -> FDLL4148; footprint Diode_SMD:D_0805_2012Metric_Pad1.15x1.40mm_HandSolder -> Diode_SMD:D_MiniMELF_Handsoldering
- D153: renamed from D152; value DIODE -> FDLL4148; footprint Diode_SMD:D_0805_2012Metric_Pad1.15x1.40mm_HandSolder -> Diode_SMD:D_MiniMELF_Handsoldering
- D154: renamed from D153; value DIODE -> FDLL4148; footprint Diode_SMD:D_0805_2012Metric_Pad1.15x1.40mm_HandSolder -> Diode_SMD:D_MiniMELF_Handsoldering
- D155: renamed from D154; value DIODE -> FDLL4148; footprint Diode_SMD:D_0805_2012Metric_Pad1.15x1.40mm_HandSolder -> Diode_SMD:D_MiniMELF_Handsoldering
- D156: renamed from D155; value DIODE -> FDLL4148; footprint Diode_SMD:D_0805_2012Metric_Pad1.15x1.40mm_HandSolder -> Diode_SMD:D_MiniMELF_Handsoldering
- D157: renamed from D156; value DIODE -> FDLL4148; footprint Diode_SMD:D_0805_2012Metric_Pad1.15x1.40mm_HandSolder -> Diode_SMD:D_MiniMELF_Handsoldering
- D158: renamed from D157; value DIODE -> FDLL4148; footprint Diode_SMD:D_0805_2012Metric_Pad1.15x1.40mm_HandSolder -> Diode_SMD:D_MiniMELF_Handsoldering
- D159: renamed from D158; value DIODE -> FDLL4148; footprint Diode_SMD:D_0805_2012Metric_Pad1.15x1.40mm_HandSolder -> Diode_SMD:D_MiniMELF_Handsoldering
- D160: renamed from D159; value DIODE -> FDLL4148; footprint Diode_SMD:D_0805_2012Metric_Pad1.15x1.40mm_HandSolder -> Diode_SMD:D_MiniMELF_Handsoldering
- D161: renamed from D160; value DIODE -> FDLL4148; footprint Diode_SMD:D_0805_2012Metric_Pad1.15x1.40mm_HandSolder -> Diode_SMD:D_MiniMELF_Handsoldering
- D33: renamed from D?; value DIODE -> FDLL4148; footprint Diode_SMD:D_0805_2012Metric_Pad1.15x1.40mm_HandSolder -> Diode_SMD:D_MicroMELF_Hadsoldering
- D34: renamed from D33; value LED -> LTST-C150KFKT; footprint LED_SMD:LED_Cree-PLCC4_3.2x2.8mm_CCW -> LED_SMD:LED_1206_3216Metric_Pad1.42x1.75mm_HandSolder
- D35: renamed from D34; value LED -> LTST-C150KFKT; footprint LED_SMD:LED_Cree-PLCC4_3.2x2.8mm_CCW -> LED_SMD:LED_1206_3216Metric_Pad1.42x1.75mm_HandSolder
- D36: renamed from D35; value LED -> LTST-C150KFKT; footprint LED_SMD:LED_Cree-PLCC4_3.2x2.8mm_CCW -> LED_SMD:LED_1206_3216Metric_Pad1.42x1.75mm_HandSolder
- D37: renamed from D36; value LED -> LTST-C150KFKT; footprint LED_SMD:LED_Cree-PLCC4_3.2x2.8mm_CCW -> LED_SMD:LED_1206_3216Metric_Pad1.42x1.75mm_HandSolder
- D38: renamed from D37; value LED -> LTST-C150KFKT; footprint LED_SMD:LED_Cree-PLCC4_3.2x2.8mm_CCW -> LED_SMD:LED_1206_3216Metric_Pad1.42x1.75mm_HandSolder
- D39: renamed from D38; value LED -> LTST-C150KFKT; footprint LED_SMD:LED_Cree-PLCC4_3.2x2.8mm_CCW -> LED_SMD:LED_1206_3216Metric_Pad1.42x1.75mm_HandSolder
- D40: renamed from D39; value LED -> LTST-C150KFKT; footprint LED_SMD:LED_Cree-PLCC4_3.2x2.8mm_CCW -> LED_SMD:LED_1206_3216Metric_Pad1.42x1.75mm_HandSolder
- D41: renamed from D40; value LED -> LTST-C150KFKT; footprint LED_SMD:LED_Cree-PLCC4_3.2x2.8mm_CCW -> LED_SMD:LED_1206_3216Metric_Pad1.42x1.75mm_HandSolder
- D42: renamed from D41; value LED -> LTST-C150KFKT; footprint LED_SMD:LED_Cree-PLCC4_3.2x2.8mm_CCW -> LED_SMD:LED_1206_3216Metric_Pad1.42x1.75mm_HandSolder
- D43: renamed from D42; value LED -> LTST-C150KFKT; footprint LED_SMD:LED_Cree-PLCC4_3.2x2.8mm_CCW -> LED_SMD:LED_1206_3216Metric_Pad1.42x1.75mm_HandSolder
- D44: renamed from D43; value LED -> LTST-C150KFKT; footprint LED_SMD:LED_Cree-PLCC4_3.2x2.8mm_CCW -> LED_SMD:LED_1206_3216Metric_Pad1.42x1.75mm_HandSolder
- D45: renamed from D44; value LED -> LTST-C150KFKT; footprint LED_SMD:LED_Cree-PLCC4_3.2x2.8mm_CCW -> LED_SMD:LED_1206_3216Metric_Pad1.42x1.75mm_HandSolder
- D46: renamed from D45; value LED -> LTST-C150KFKT; footprint LED_SMD:LED_Cree-PLCC4_3.2x2.8mm_CCW -> LED_SMD:LED_1206_3216Metric_Pad1.42x1.75mm_HandSolder
- D47: renamed from D46; value LED -> LTST-C150KFKT; footprint LED_SMD:LED_Cree-PLCC4_3.2x2.8mm_CCW -> LED_SMD:LED_1206_3216Metric_Pad1.42x1.75mm_HandSolder
- D48: renamed from D47; value LED -> LTST-C150KFKT; footprint LED_SMD:LED_Cree-PLCC4_3.2x2.8mm_CCW -> LED_SMD:LED_1206_3216Metric_Pad1.42x1.75mm_HandSolder
- D49: renamed from D48; value LED -> LTST-C150KFKT; footprint LED_SMD:LED_Cree-PLCC4_3.2x2.8mm_CCW -> LED_SMD:LED_1206_3216Metric_Pad1.42x1.75mm_HandSolder
- D50: renamed from D49; value LED -> LTST-C150KFKT; footprint LED_SMD:LED_Cree-PLCC4_3.2x2.8mm_CCW -> LED_SMD:LED_1206_3216Metric_Pad1.42x1.75mm_HandSolder
- D51: renamed from D50; value LED -> LTST-C150KFKT; footprint LED_SMD:LED_Cree-PLCC4_3.2x2.8mm_CCW -> LED_SMD:LED_1206_3216Metric_Pad1.42x1.75mm_HandSolder
- D52: renamed from D51; value LED -> LTST-C150KFKT; footprint LED_SMD:LED_Cree-PLCC4_3.2x2.8mm_CCW -> LED_SMD:LED_1206_3216Metric_Pad1.42x1.75mm_HandSolder
- D53: renamed from D52; value LED -> LTST-C150KFKT; footprint LED_SMD:LED_Cree-PLCC4_3.2x2.8mm_CCW -> LED_SMD:LED_1206_3216Metric_Pad1.42x1.75mm_HandSolder
- D54: renamed from D53; value LED -> LTST-C150KFKT; footprint LED_SMD:LED_Cree-PLCC4_3.2x2.8mm_CCW -> LED_SMD:LED_1206_3216Metric_Pad1.42x1.75mm_HandSolder
- D55: renamed from D54; value LED -> LTST-C150KFKT; footprint LED_SMD:LED_Cree-PLCC4_3.2x2.8mm_CCW -> LED_SMD:LED_1206_3216Metric_Pad1.42x1.75mm_HandSolder
- D56: renamed from D55; value LED -> LTST-C150KFKT; footprint LED_SMD:LED_Cree-PLCC4_3.2x2.8mm_CCW -> LED_SMD:LED_1206_3216Metric_Pad1.42x1.75mm_HandSolder
- D57: renamed from D56; value LED -> LTST-C150KFKT; footprint LED_SMD:LED_Cree-PLCC4_3.2x2.8mm_CCW -> LED_SMD:LED_1206_3216Metric_Pad1.42x1.75mm_HandSolder
- D58: renamed from D57; value LED -> LTST-C150KFKT; footprint LED_SMD:LED_Cree-PLCC4_3.2x2.8mm_CCW -> LED_SMD:LED_1206_3216Metric_Pad1.42x1.75mm_HandSolder
- D59: renamed from D58; value LED -> LTST-C150KFKT; footprint LED_SMD:LED_Cree-PLCC4_3.2x2.8mm_CCW -> LED_SMD:LED_1206_3216Metric_Pad1.42x1.75mm_HandSolder
- D60: renamed from D59; value LED -> LTST-C150KFKT; footprint LED_SMD:LED_Cree-PLCC4_3.2x2.8mm_CCW -> LED_SMD:LED_1206_3216Metric_Pad1.42x1.75mm_HandSolder
- D61: renamed from D60; value LED -> LTST-C150KFKT; footprint LED_SMD:LED_Cree-PLCC4_3.2x2.8mm_CCW -> LED_SMD:LED_1206_3216Metric_Pad1.42x1.75mm_HandSolder
- D62: renamed from D61; value LED -> LTST-C150KFKT; footprint LED_SMD:LED_Cree-PLCC4_3.2x2.8mm_CCW -> LED_SMD:LED_1206_3216Metric_Pad1.42x1.75mm_HandSolder
- D63: renamed from D62; value LED -> LTST-C150KFKT; footprint LED_SMD:LED_Cree-PLCC4_3.2x2.8mm_CCW -> LED_SMD:LED_1206_3216Metric_Pad1.42x1.75mm_HandSolder
- D64: renamed from D63; value LED -> LTST-C150KFKT; footprint LED_SMD:LED_Cree-PLCC4_3.2x2.8mm_CCW -> LED_SMD:LED_1206_3216Metric_Pad1.42x1.75mm_HandSolder
- D65: renamed from D64; value LED -> LTST-C150KFKT; footprint LED_SMD:LED_Cree-PLCC4_3.2x2.8mm_CCW -> LED_SMD:LED_1206_3216Metric_Pad1.42x1.75mm_HandSolder
- D66: renamed from D65; value LED -> LTST-C150KFKT; footprint LED_SMD:LED_Cree-PLCC4_3.2x2.8mm_CCW -> LED_SMD:LED_1206_3216Metric_Pad1.42x1.75mm_HandSolder
- D67: renamed from D66; value LED -> LTST-C150KFKT; footprint LED_SMD:LED_Cree-PLCC4_3.2x2.8mm_CCW -> LED_SMD:LED_1206_3216Metric_Pad1.42x1.75mm_HandSolder
- D68: renamed from D67; value LED -> LTST-C150KFKT; footprint LED_SMD:LED_Cree-PLCC4_3.2x2.8mm_CCW -> LED_SMD:LED_1206_3216Metric_Pad1.42x1.75mm_HandSolder
- D69: renamed from D68; value LED -> LTST-C150KFKT; footprint LED_SMD:LED_Cree-PLCC4_3.2x2.8mm_CCW -> LED_SMD:LED_1206_3216Metric_Pad1.42x1.75mm_HandSolder
- D70: renamed from D69; value LED -> LTST-C150KFKT; footprint LED_SMD:LED_Cree-PLCC4_3.2x2.8mm_CCW -> LED_SMD:LED_1206_3216Metric_Pad1.42x1.75mm_HandSolder
- D71: renamed from D70; value LED -> LTST-C150KFKT; footprint LED_SMD:LED_Cree-PLCC4_3.2x2.8mm_CCW -> LED_SMD:LED_1206_3216Metric_Pad1.42x1.75mm_HandSolder
- D72: renamed from D71; value LED -> LTST-C150KFKT; footprint LED_SMD:LED_Cree-PLCC4_3.2x2.8mm_CCW -> LED_SMD:LED_1206_3216Metric_Pad1.42x1.75mm_HandSolder
- D73: renamed from D72; value LED -> LTST-C150KFKT; footprint LED_SMD:LED_Cree-PLCC4_3.2x2.8mm_CCW -> LED_SMD:LED_1206_3216Metric_Pad1.42x1.75mm_HandSolder
- D74: renamed from D73; value LED -> LTST-C150KFKT; footprint LED_SMD:LED_Cree-PLCC4_3.2x2.8mm_CCW -> LED_SMD:LED_1206_3216Metric_Pad1.42x1.75mm_HandSolder
- D75: renamed from D74; value LED -> LTST-C150KFKT; footprint LED_SMD:LED_Cree-PLCC4_3.2x2.8mm_CCW -> LED_SMD:LED_1206_3216Metric_Pad1.42x1.75mm_HandSolder
- D76: renamed from D75; value LED -> LTST-C150KFKT; footprint LED_SMD:LED_Cree-PLCC4_3.2x2.8mm_CCW -> LED_SMD:LED_1206_3216Metric_Pad1.42x1.75mm_HandSolder
- D77: renamed from D76; value LED -> LTST-C150KFKT; footprint LED_SMD:LED_Cree-PLCC4_3.2x2.8mm_CCW -> LED_SMD:LED_1206_3216Metric_Pad1.42x1.75mm_HandSolder
- D78: renamed from D77; value LED -> LTST-C150KFKT; footprint LED_SMD:LED_Cree-PLCC4_3.2x2.8mm_CCW -> LED_SMD:LED_1206_3216Metric_Pad1.42x1.75mm_HandSolder
- D79: renamed from D78; value LED -> LTST-C150KFKT; footprint LED_SMD:LED_Cree-PLCC4_3.2x2.8mm_CCW -> LED_SMD:LED_1206_3216Metric_Pad1.42x1.75mm_HandSolder
- D80: renamed from D79; value LED -> LTST-C150KFKT; footprint LED_SMD:LED_Cree-PLCC4_3.2x2.8mm_CCW -> LED_SMD:LED_1206_3216Metric_Pad1.42x1.75mm_HandSolder
- D81: renamed from D80; value LED -> LTST-C150KFKT; footprint LED_SMD:LED_Cree-PLCC4_3.2x2.8mm_CCW -> LED_SMD:LED_1206_3216Metric_Pad1.42x1.75mm_HandSolder
- D82: renamed from D81; value DIODE -> FDLL4148; footprint Diode_SMD:D_0805_2012Metric_Pad1.15x1.40mm_HandSolder -> Diode_SMD:D_MiniMELF_Handsoldering
- D83: renamed from D82; value DIODE -> FDLL4148; footprint Diode_SMD:D_0805_2012Metric_Pad1.15x1.40mm_HandSolder -> Diode_SMD:D_MiniMELF_Handsoldering
- D84: renamed from D83; value DIODE -> FDLL4148; footprint Diode_SMD:D_0805_2012Metric_Pad1.15x1.40mm_HandSolder -> Diode_SMD:D_MiniMELF_Handsoldering
- D85: renamed from D84; value DIODE -> FDLL4148; footprint Diode_SMD:D_0805_2012Metric_Pad1.15x1.40mm_HandSolder -> Diode_SMD:D_MiniMELF_Handsoldering
- D86: renamed from D85; value DIODE -> FDLL4148; footprint Diode_SMD:D_0805_2012Metric_Pad1.15x1.40mm_HandSolder -> Diode_SMD:D_MiniMELF_Handsoldering
- D87: renamed from D86; value DIODE -> FDLL4148; footprint Diode_SMD:D_0805_2012Metric_Pad1.15x1.40mm_HandSolder -> Diode_SMD:D_MiniMELF_Handsoldering
- D88: renamed from D87; value DIODE -> FDLL4148; footprint Diode_SMD:D_0805_2012Metric_Pad1.15x1.40mm_HandSolder -> Diode_SMD:D_MiniMELF_Handsoldering
- D89: renamed from D88; value DIODE -> FDLL4148; footprint Diode_SMD:D_0805_2012Metric_Pad1.15x1.40mm_HandSolder -> Diode_SMD:D_MiniMELF_Handsoldering
- D90: renamed from D89; value DIODE -> FDLL4148; footprint Diode_SMD:D_0805_2012Metric_Pad1.15x1.40mm_HandSolder -> Diode_SMD:D_MiniMELF_Handsoldering
- D91: renamed from D90; value DIODE -> FDLL4148; footprint Diode_SMD:D_0805_2012Metric_Pad1.15x1.40mm_HandSolder -> Diode_SMD:D_MiniMELF_Handsoldering
- D92: renamed from D91; value DIODE -> FDLL4148; footprint Diode_SMD:D_0805_2012Metric_Pad1.15x1.40mm_HandSolder -> Diode_SMD:D_MiniMELF_Handsoldering
- D93: renamed from D92; value DIODE -> FDLL4148; footprint Diode_SMD:D_0805_2012Metric_Pad1.15x1.40mm_HandSolder -> Diode_SMD:D_MiniMELF_Handsoldering
- D94: renamed from D93; value DIODE -> FDLL4148; footprint Diode_SMD:D_0805_2012Metric_Pad1.15x1.40mm_HandSolder -> Diode_SMD:D_MiniMELF_Handsoldering
- D95: renamed from D94; value DIODE -> FDLL4148; footprint Diode_SMD:D_0805_2012Metric_Pad1.15x1.40mm_HandSolder -> Diode_SMD:D_MiniMELF_Handsoldering
- D96: renamed from D95; value DIODE -> FDLL4148; footprint Diode_SMD:D_0805_2012Metric_Pad1.15x1.40mm_HandSolder -> Diode_SMD:D_MiniMELF_Handsoldering
- D97: renamed from D96; value DIODE -> FDLL4148; footprint Diode_SMD:D_0805_2012Metric_Pad1.15x1.40mm_HandSolder -> Diode_SMD:D_MiniMELF_Handsoldering
- D98: renamed from D97; value DIODE -> FDLL4148; footprint Diode_SMD:D_0805_2012Metric_Pad1.15x1.40mm_HandSolder -> Diode_SMD:D_MiniMELF_Handsoldering
- D99: renamed from D98; value DIODE -> FDLL4148; footprint Diode_SMD:D_0805_2012Metric_Pad1.15x1.40mm_HandSolder -> Diode_SMD:D_MiniMELF_Handsoldering
- POT1, POT2: value 10kE -> 10KE; footprint digikey-footprints:Trimpot_3.8mmx3.6mm_TC33X-2-103E -> Connector_PinHeader_2.54mm:PinHeader_1x03_P2.54mm_Horizontal
- Q1, Q2: footprint digikey-footprints:SOIC-18_W7.5mm -> Package_SO:SOIC-18W_7.5x11.6mm_P1.27mm
- R1, R2, R3, R4, R5: value R -> 47E; footprint Resistor_SMD:R_0805_2012Metric_Pad1.15x1.40mm_HandSolder -> Resistor_SMD:R_1206_3216Metric_Pad1.42x1.75mm_HandSolder
- R10: renamed from R8; footprint Resistor_SMD:R_0805_2012Metric_Pad1.15x1.40mm_HandSolder -> Resistor_SMD:R_1206_3216Metric_Pad1.42x1.75mm_HandSolder
- R11, R16, R7, R8, R9: renamed from R?; value R -> 10K; footprint Resistor_SMD:R_0805_2012Metric_Pad1.15x1.40mm_HandSolder -> Resistor_SMD:R_1206_3216Metric_Pad1.42x1.75mm_HandSolder
- R12: renamed from R9; footprint Resistor_SMD:R_0805_2012Metric_Pad1.15x1.40mm_HandSolder -> Resistor_SMD:R_1206_3216Metric_Pad1.42x1.75mm_HandSolder
- R13: renamed from R11; footprint Resistor_SMD:R_0805_2012Metric_Pad1.15x1.40mm_HandSolder -> Resistor_SMD:R_1206_3216Metric_Pad1.42x1.75mm_HandSolder
- R14: renamed from R10; footprint Resistor_SMD:R_0805_2012Metric_Pad1.15x1.40mm_HandSolder -> Resistor_SMD:R_1206_3216Metric_Pad1.42x1.75mm_HandSolder
- R15: renamed from R12; footprint Resistor_SMD:R_0805_2012Metric_Pad1.15x1.40mm_HandSolder -> Resistor_SMD:R_1206_3216Metric_Pad1.42x1.75mm_HandSolder
- R6: value R -> 1K; footprint Resistor_SMD:R_0805_2012Metric_Pad1.15x1.40mm_HandSolder -> Resistor_SMD:R_1206_3216Metric_Pad1.42x1.75mm_HandSolder
- S1, S10, S11, S12, S13, S14, S15, S16, S17, S18, S19, S2, S20, S21, S22, S23, S24, S25, S26, S27, S28, S29, S3, S30, S31, S32, S33, S34, S35, S36, S37, S38, S39, S4, S40, S41, S42, S43, S44, S45, S46, S47, S48, S49, S5, S50, S51, S52, S53, S54, S55, S56, S57, S58, S59, S6, S60, S61, S62, S63, S64, S65, S66, S67, S68, S69, S7, S70, S71, S72, S73, S74, S75, S76, S77, S78, S79, S8, S80, S9: footprint digikey-footprints:PushButton_12x12mm_THT_GPTS203211B -> digikey-footprints:Switch_Tactile_SMD_6x6mm
- U2, U5: value 4017 -> CD74HC4017; footprint (none) -> Package_SO:SOIC-16_3.9x9.9mm_P1.27mm
- U7: footprint digikey-footprints:SSOP-16_W3.90mm -> pieter:FT230XS-HEADER
- renumbered J2 to J13, U4 to U3
Connections:
- wire segments 638 -> 627
- no-connect marks 76 -> 89
Other:
- note added: "NOTE THAT THIS CHIP IS MISSING \nSOME CONNECTIONS AS THESE \nARE PRESENT ON THE BOARD BEING \nUSED FROM ED315"
- note added: "TESTING HEADERS"

Commit message: Updated footprint link with symbols; Started PCB Design - completed button/led array.
Parts:
- POT1, POT2: footprint Connector_PinHeader_2.54mm:PinHeader_1x03_P2.54mm_Horizontal -> Connector_PinHeader_2.54mm:PinHeader_1x03_P2.54mm_Vertical
- S1, S10, S11, S12, S13, S14, S15, S16, S17, S18, S19, S2, S20, S21, S22, S23, S24, S25, S26, S27, S28, S29, S3, S30, S31, S32, S33, S34, S35, S36, S37, S38, S39, S4, S40, S41, S42, S43, S44, S45, S46, S47, S48, S49, S5, S50, S51, S52, S53, S54, S55, S56, S57, S58, S59, S6, S60, S61, S62, S63, S64, S65, S66, S67, S68, S69, S7, S70, S71, S72, S73, S74, S75, S76, S77, S78, S79, S8, S80, S9: footprint digikey-footprints:Switch_Tactile_SMD_6x6mm -> pieter:Switch_Tactile_SMD_6x6mm
Connections:
- net labels removed: bv7
